File: STM32G491RE.kicad_pcb (KiCad board)
At the start: 2 copper layers, 207.9 x 155.8 mm, 202 parts, among them J4 OLED I2C, J5 BAT VIN, J6 TYPE-C_16PIN_2MD__073_, J7 Battery, Q1 PMOS, Q10 IBLML6344, Q11 IBLML6344, Q2 PMOS, Q3 PMOS, Q4 IBLML6344, Q5 BC817-40, Q6 BC817-40, Q7 IBLML6344, Q8 BC817-40, Q9 BC817-40, U1 TPS564257DRLR, U10 ESP32-S3-MINI-1-N8, U2 STM32G491RETx, U3 TPS2113ADRBR, U4 DRV8835DSSR, U5 M24M02-DRMN6TP, U6 MP2639A, U7 TPS79601DRBR, U8 LMV331M5, U9 LMV331M5, Y1 24MHz, Y2 32.768KHz

Commit message: slightly change schematic, making sure everything is ok, preparing for finalization
Parts:
- added Ce1: 100nF, Capacitor_SMD:C_0805_2012Metric_Pad1.18x1.45mm_HandSolder, F.Cu at (39.1, 47.4)
- added J11: Conn_01x04, Connector_PinHeader_2.54mm:PinHeader_1x04_P2.54mm_Vertical, F.Cu at (29.1, 106.8)
- added J12: Conn_01x04, Connector_PinHeader_2.54mm:PinHeader_1x04_P2.54mm_Vertical, F.Cu at (113.3, 107.5)
- added J9: Conn_01x06, Connector_PinHeader_2.54mm:PinHeader_1x06_P2.54mm_Vertical, F.Cu at (86.5, 105.7)
- added R56: 2k, Resistor_SMD:R_0805_2012Metric_Pad1.20x1.40mm_HandSolder, F.Cu at (43.8, 47.3)
- added SW1: switch, Button_Switch_SMD:Nidec_Copal_CAS-120A, F.Cu at (50.9, 42.9)
- added U11: TSOP38238, kicad_custom:TSOP382, F.Cu at (39.2, 41.4)
- BTN7, C44, C45, C61, C62, L3, R27, U10: moved to B.Cu
- J4: footprint Connector_PinSocket_2.54mm:PinSocket_2x04_P2.54mm_Horizontal -> Connector_PinSocket_2.54mm:PinSocket_2x04_P2.54mm_Vertical
- moved BTN7 116.8 mm to (74.9, 146.4), turned to 0 degrees
- moved J4 112.5 mm to (43.3, 160.3), turned to 90 degrees
- moved C62 109.8 mm to (78.9, 146.5)
- moved R27 106.3 mm to (80.9, 146.5)
- moved C7 105.1 mm to (90.5, 144.1), turned to -90 degrees
- moved C11 100.1 mm to (86.5, 142.9), turned to -90 degrees
- moved C10 95.4 mm to (92.8, 137.7), turned to 90 degrees
- moved U4 93.8 mm to (86.1, 139.7), turned to -90 degrees
- moved C9 93.5 mm to (90.7, 137.8), turned to 90 degrees
- moved C8 91.8 mm to (88.6, 137.7), turned to 90 degrees
- moved U10 91.6 mm to (89.8, 153.2), turned to 180 degrees
- moved C12 84.9 mm to (87.9, 134.3), turned to 180 degrees
- moved C13 82.1 mm to (83.7, 134.3), turned to 180 degrees
- moved BTN8 81.0 mm to (63.0, 102.2)
- moved C5 81.0 mm to (64.0, 99.2)
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Connections:
- C60 pad 2: V_DIODE -> Net-(D12-K)
- C72 pad 2: V_DIODE -> Net-(D15-K)
- D12 pad 1: V_DIODE -> Net-(D12-K)
- D12 pad 2: Signal out -> Signal out_LU
- D15 pad 1: V_DIODE -> Net-(D15-K)
- D15 pad 2: Signal out -> Signal out_R
- D16 pad 1: V_DIODE -> Net-(D15-K)
- D16 pad 2: Signal out -> Signal out_RU
- D9 pad 1: V_DIODE -> Net-(D12-K)
- D9 pad 2: Signal out -> Signal out_L
- Q1 pad D: Net-(J5-Pin_2) -> Net-(SW1-C)
- R11 pad 2: V_DIODE -> Net-(D12-K)
- R28 pad 1: Signal out -> Signal out_L
- R36 pad 1: Gate ctrl -> Gate ctrl_L
- R52 pad 1: Gate ctrl -> Gate ctrl_LU
- R57 pad 1: Signal out -> Signal out_LU
- R58 pad 1: Gate ctrl -> Gate ctrl_R
- R59 pad 1: Gate ctrl -> Gate ctrl_RU
- R66 pad 2: V_DIODE -> Net-(D15-K)
- R68 pad 1: Signal out -> Signal out_R
- R69 pad 1: Signal out -> Signal out_RU
Other:
- board text added: "BMS"
- board text added: "CONNECTORS"
- board text added: "STEP DOWNS"
- board text added: "USB"
